File: USB-Flash-Drive/USB-Flash-Drive.kicad_sch (KiCad schematic)
At the start: 37 parts, among them J1 USB_A, J2 Conn_01x03_Pin, U1 RP2040, U2 W25Q128JVS, U3 AMS1117, U4 W25N01GVZEIG, Y2 ABM8-272-T3

Commit message: update flash-drive to KiCAD 9.0
Changed lines of the file:
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@@
 (kicad_sch
-	(version 20231120)
+	(version 20250114)
 	(generator "eeschema")
-	(generator_version "8.0")
+	(generator_version "9.0")
 	(paper "A4")
 	(junction
@@
 	(label "DEBUG_GND"
 		(at 129.54 92.71 270)
-		(fields_autoplaced yes)
 		(effects
 			(font
@@
 	(label "SPI_COPI"
 		(at 144.78 130.81 180)
-		(fields_autoplaced yes)
 		(effects
 			(font
@@
 	(label "SPI_CLK"
 		(at 144.78 128.27 180)
-		(fields_autoplaced yes)
 		(effects
 			(font
@@
 	(label "SPI_CLK"
 		(at 118.11 130.81 0)
-		(fields_autoplaced yes)
 		(effects
 			(font
@@
 	(label "XOUT"
 		(at 60.96 142.24 180)
-		(fields_autoplaced yes)
 		(effects
 			(font
@@
 	(label "SPI_COPI"
 		(at 118.11 133.35 0)
-		(fields_autoplaced yes)
 		(effects
 			(font
@@
 	(label "RESET"
 		(at 66.04 85.09 270)
-		(fields_autoplaced yes)
 		(effects
 			(font
@@
 	(label "SPI_CIPO"
 		(at 118.11 125.73 0)
-		(fields_autoplaced yes)
 		(effects
 			(font
@@
 	(label "XIN"
 		(at 55.88 130.81 0)
-		(fields_autoplaced yes)
 		(effects
 			(font
@@
 	(label "SPI_CIPO"
 		(at 144.78 133.35 180)
-		(fields_autoplaced yes)
 		(effects
 			(font
@@
 	(label "SPI_CS"
 		(at 144.78 125.73 180)
-		(fields_autoplaced yes)
 		(effects
 			(font
@@
 	(label "BOOT"
 		(at 152.4 91.44 90)
-		(fields_autoplaced yes)
 		(effects
 			(font
@@
 	(label "SPI_CS"
 		(at 118.11 128.27 0)
-		(fields_autoplaced yes)
 		(effects
 			(font
@@
 		)
 	)
+	(embedded_fonts no)
 )
