File: RPU1.1-Controller/RPU1.1-Controller.kicad_pcb (KiCad board)
At the start: 2 copper layers, 100.3 x 75.5 mm, 124 parts, among them P0 Pressure Transducer, P1 Pressure Transducer, P2 Pressure Transducer, P3 Pressure Transducer, P4 Pressure Transducer, P5 Pressure Transducer, Q1 S8550, Q2 IRLZ44N, Q3 IRLZ44N, Q4 IRLZ44N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

Commit message: A bunch of KiCad Projects
Routing:
- net GND: vias 21 -> 75
